File: RADSAT-SK Timer/_saved_RADSAT-SK Timer 2.sch (KiCad schematic (older format))
At the start: 29 parts, among them J201 Conn_01x04, J202 USB_B_Micro, J203 Conn_01x02, J204 Conn_01x02, J205 Conn_01x02, J206 Conn_01x02, J207 Conn_01x02, Q201 IRLML2060, SW201 SW_Push, SW202 SW_Push, SW203 SW_Push, SW204 SW_Push, SW205 SW_Push, SW206 SW_Push, U202 LTC3440EMSPBF

Commit message: Schematic: Added- 2 more inhibit ports Added- RBF Ports In and Out Connected USb Charger to connector H1-32. Layout: Port positioning and adjustments to some existing circuitry for better tracing.
Parts:
- renumbered Q201 to Q202
Changed lines of the file:
@@
 P 4700 3675
 AR Path="/60E15E10" Ref="Q?"  Part="1"
-AR Path="/602E25D3/60E15E10" Ref="Q201"  Part="1"
-F 0 "Q201" H 4475 3600 50  0000 L CNN
+AR Path="/602E25D3/60E15E10" Ref="Q202"  Part="1"
+F 0 "Q202" H 4475 3600 50  0000 L CNN
 F 1 "IRLML2060" H 4375 3500 50  0000 L CNN
 F 2 "Package_TO_SOT_SMD:SOT-23" H 4900 3600 50  0001 L CIN
 F 3 "https://www.infineon.com/dgdl/irlml2060pbf.pdf?fileId=5546d462533600a401535664b7fb25ee" H 4700 3675 50  0001 L CNN
 	1    4700 3675
-	1    0    0    -1
+	1    0    0    1
 $EndComp
 Wire Wire Line
@@
 Connection ~ 3275 3675
 $Comp
-L power:GND #PWR?
+L power:GND #PWR0106
 U 1 1 60E611EF
 P 2725 4175
-F 0 "#PWR?" H 2725 3925 50  0001 C CNN
+F 0 "#PWR0106" H 2725 3925 50  0001 C CNN
 F 1 "GND" H 2730 4002 50  0000 C CNN
 F 2 "" H 2725 4175 50  0001 C CNN
@@
 NoConn ~ 1625 5675
 $Comp
-L power:GND #PWR?
+L power:GND #PWR0108
 U 1 1 60E8A087
 P 1325 6050
-F 0 "#PWR?" H 1325 5800 50  0001 C CNN
+F 0 "#PWR0108" H 1325 5800 50  0001 C CNN
 F 1 "GND" H 1330 5877 50  0000 C CNN
 F 2 "" H 1325 6050 50  0001 C CNN
