File: RADSAT-SK Timer/_autosave-RADSAT-SK Timer 2.sch (KiCad schematic (older format))
At the start: 36 parts, among them J201 Conn_01x04, J202 USB_B_Micro, J203 Conn_01x02, J204 Conn_01x02, J205 Conn_01x02, J206 Conn_01x02, J207 Conn_01x02, J208 Conn_01x05_Male, Q201 IRLML2060, Q202 IRLML2060, SW201 SW_Push, SW202 SW_Push, SW203 SW_Push, SW204 SW_Push, SW205 SW_Push, SW206 SW_Push, U202 LTC3440EMSPBF

Commit message: Mason has updated some footprints
Parts:
- BT1: renamed from BT?; footprint (none) -> Battery:BatteryHolder_Keystone_1060_1x2032
- Q1: renamed from Q?; footprint (none) -> Package_TO_SOT_SMD:SOT-23
- R1, R2: renamed from R?; footprint (none) -> Resistor_SMD:R_0805_2012Metric
- gave numbers to parts that had none: 2
Changed lines of the file:
@@
 Wire Wire Line
 	9925 1425 9550 1425
-Connection ~ 9550 1425
 Wire Wire Line
 	9100 2025 9925 2025
@@
 	6425 5000 6425 7800
 $Comp
-L Device:R R?
+L Device:R R1
 U 1 1 611EADEE
 P 3600 6050
-F 0 "R?" H 3670 6096 50  0000 L CNN
+F 0 "R1" H 3670 6096 50  0000 L CNN
 F 1 "R" H 3670 6005 50  0000 L CNN
-F 2 "" V 3530 6050 50  0001 C CNN
+F 2 "Resistor_SMD:R_0805_2012Metric" V 3530 6050 50  0001 C CNN
 F 3 "~" H 3600 6050 50  0001 C CNN
 	1    3600 6050
@@
 $EndComp
 $Comp
-L Diode:5KPxxA D?
+L Diode:5KPxxA D1
 U 1 1 611ED310
 P 4000 6050
-F 0 "D?" V 3954 6130 50  0000 L CNN
+F 0 "D1" V 3954 6130 50  0000 L CNN
 F 1 "5KPxxA" V 4045 6130 50  0000 L CNN
 F 2 "Diode_THT:D_P600_R-6_P20.00mm_Horizontal" H 4000 5850 50  0001 C CNN
@@
 $EndComp
 $Comp
-L Device:R R?
+L Device:R R2
 U 1 1 611EE061
 P 4500 5900
-F 0 "R?" V 4293 5900 50  0000 C CNN
+F 0 "R2" V 4293 5900 50  0000 C CNN
 F 1 "R" V 4384 5900 50  0000 C CNN
-F 2 "" V 4430 5900 50  0001 C CNN
+F 2 "Resistor_SMD:R_0805_2012Metric" V 4430 5900 50  0001 C CNN
 F 3 "~" H 4500 5900 50  0001 C CNN
 	1    4500 5900
@@
 $EndComp
 $Comp
-L Device:Q_NMOS_DGS Q?
+L Device:Q_NMOS_DGS Q1
 U 1 1 611F24A8
 P 4975 5900
-F 0 "Q?" H 5179 5946 50  0000 L CNN
+F 0 "Q1" H 5179 5946 50  0000 L CNN
 F 1 "Q_NMOS_DGS" H 5179 5855 50  0000 L CNN
-F 2 "" H 5175 6000 50  0001 C CNN
+F 2 "Package_TO_SOT_SMD:SOT-23" H 5175 6000 50  0001 C CNN
 F 3 "~" H 4975 5900 50  0001 C CNN
 	1    4975 5900
@@
 DETECT LOGIC FOR RBF
 $Comp
-L Device:Battery_Cell BT?
+L Device:Battery_Cell BT1
 U 1 1 611F46E7
 P 4225 5375
-F 0 "BT?" H 4343 5471 50  0000 L CNN
+F 0 "BT1" H 4343 5471 50  0000 L CNN
 F 1 "Battery_Cell" H 4343 5380 50  0000 L CNN
-F 2 "" V 4225 5435 50  0001 C CNN
+F 2 "Battery:BatteryHolder_Keystone_1060_1x2032" V 4225 5435 50  0001 C CNN
 F 3 "~" V 4225 5435 50  0001 C CNN
 	1    4225 5375
@@
 	3900 5175 3900 5700
 $Comp
-L Connector:Conn_01x02_Male J?
+L Connector:Conn_01x02_Male J1
 U 1 1 6126FDD8
 P 5300 5275
-F 0 "J?" H 5272 5157 50  0000 R CNN
+F 0 "J1" H 5272 5157 50  0000 R CNN
 F 1 "Conn_01x02_Male" H 5272 5248 50  0000 R CNN
 F 2 "Connector_Molex:Molex_PicoBlade_53047-0210_1x02_P1.25mm_Vertical" H 5300 5275 50  0001 C CNN
@@
 	3600 6200 4000 6200
 $Comp
-L power:GND #PWR?
+L power:GND #PWR0117
 U 1 1 6129EA2C
 P 5075 6200
-F 0 "#PWR?" H 5075 5950 50  0001 C CNN
+F 0 "#PWR0117" H 5075 5950 50  0001 C CNN
 F 1 "GND" H 5080 6027 50  0001 C CNN
 F 2 "" H 5075 6200 50  0001 C CNN
