File: RADSAT-SK Timer/_autosave-RADSAT-SK Timer.sch (KiCad schematic (older format))
At the start: 71 parts, among them J101 Conn_02x26_Odd_Even, J103 Conn_02x26_Odd_Even, Q101 IRLML2060, Q102 IRLML2060, Q103 IRLML2060, Q104 IRLML2060, Q105 IRLML2060, Q106 IRLML2060, Q107 IRLML2060, Q108 IRLML2060, Q109 IRLML2060, U101 LM397MF, U102 LM397MF, U103 LM397MF, U104 CD4052B

Commit message: Revert "Retrace (#8)" (#11)
This reverts commit b83679d15abd0ed1c357c8fd6e32726f91c1f504.
Parts:
- added D102: LED, LED_SMD:LED_0805_2012Metric, symbol Device:LED
- added R138: 1k, Resistor_SMD:R_0805_2012Metric, symbol Device:R
Connections:
- wire segments 230 -> 229
Changed lines of the file:
@@
 Connection ~ 3250 750
-Wire Wire Line
-	2875 750  2450 750
 Wire Wire Line
 	1300 750  1300 875
@@
 Wire Wire Line
 	8225 1075 8625 1075
-Text GLabel 7875 1275 0    50   Input ~ 0
+Text GLabel 7425 1275 0    50   Input ~ 0
 BUS_EN
 Wire Wire Line
@@
 	8050 2175 8425 2175
 Connection ~ 8425 2175
-Wire Wire Line
-	7875 1275 8050 1275
 Connection ~ 8050 1275
 Wire Wire Line
@@
 Wire Wire Line
 	8050 1675 8050 2175
-$Comp
-L power:+BATT #PWR0104
-U 1 1 601B4594
-P 2100 700
-F 0 "#PWR0104" H 2100 550 50  0001 C CNN
-F 1 "+BATT" H 2100 875 50  0000 C CNN
-F 2 "" H 2100 700 50  0001 C CNN
-F 3 "" H 2100 700 50  0001 C CNN
-	1    2100 700
-	1    0    0    -1
-$EndComp
 Wire Wire Line
 	9975 775  10625 775
@@
 Text Notes 7150 2675 0    79   ~ 0
 CSKB Connectors
-Wire Wire Line
-	2100 750  2100 700
-Connection ~ 2100 750
-Wire Wire Line
-	2100 750  1300 750
 Text Notes 525  6925 0    79   ~ 0
 Batteries, Charger, Booster, Mechanical Inhibits, Antenna Connector, Output Connectors
@@
 	3575 1125 3575 1225
 $Comp
-L power:+5V #PWR0105
-U 1 1 601A2221
-P 2450 700
-F 0 "#PWR0105" H 2450 550 50  0001 C CNN
-F 1 "+5V" H 2465 873 50  0000 C CNN
-F 2 "" H 2450 700 50  0001 C CNN
-F 3 "" H 2450 700 50  0001 C CNN
-	1    2450 700
-	1    0    0    -1
-$EndComp
-Connection ~ 2450 750
-Wire Wire Line
-	2450 750  2100 750
-Wire Wire Line
-	2450 750  2450 700
-$Comp
 L Device:R R117
 U 1 1 6023BA87
@@
 Connection ~ 3250 2850
 Wire Wire Line
-	2875 2850 2450 2850
-Wire Wire Line
 	1300 2850 1300 2975
 Connection ~ 2875 2850
@@
 	3575 3225 3575 3325
 $Comp
-L power:+5V #PWR0106
-U 1 1 6023BB60
-P 2450 2800
-F 0 "#PWR0106" H 2450 2650 50  0001 C CNN
-F 1 "+5V" H 2465 2973 50  0000 C CNN
-F 2 "" H 2450 2800 50  0001 C CNN
-F 3 "" H 2450 2800 50  0001 C CNN
-	1    2450 2800
-	1    0    0    -1
-$EndComp
-Connection ~ 2450 2850
-Wire Wire Line
-	2450 2850 2100 2850
-Wire Wire Line
-	2450 2850 2450 2800
-$Comp
 L Device:R R118
 U 1 1 60268A7A
@@
 Connection ~ 3250 4900
 Wire Wire Line
-	2875 4900 2450 4900
-Wire Wire Line
 	1300 4900 1300 5025
 Connection ~ 2875 4900
@@
 Wire Wire Line
 	3575 5275 3575 5375
-$Comp
-L power:+5V #PWR0108
-U 1 1 60268B53
-P 2450 4850
-F 0 "#PWR0108" H 2450 4700 50  0001 C CNN
-F 1 "+5V" H 2465 5023 50  0000 C CNN
-F 2 "" H 2450 4850 50  0001 C CNN
-F 3 "" H 2450 4850 50  0001 C CNN
-	1    2450 4850
-	1    0    0    -1
-$EndComp
-Connection ~ 2450 4900
-Wire Wire Line
-	2450 4900 2100 4900
-Wire Wire Line
-	2450 4900 2450 4850
 $Sheet
 S 2325 7150 1725 375
@@
 NoConn ~ 10350 4225
 NoConn ~ 10350 4125
+$Comp
+L Device:LED D102
+U 1 1 600FEA55
+P 7600 1550
+F 0 "D102" V 7639 1432 50  0000 R CNN
+F 1 "LED" V 7548 1432 50  0000 R CNN
+F 2 "LED_SMD:LED_0805_2012Metric" H 7600 1550 50  0001 C CNN
+F 3 "~" H 7600 1550 50  0001 C CNN
+	1    7600 1550
+	0    -1   -1   0
+$EndComp
+$Comp
+L Device:R R138
+U 1 1 60100324
+P 7600 1950
+F 0 "R138" H 7670 1996 50  0000 L CNN
+F 1 "1k" H 7670 1905 50  0000 L CNN
+F 2 "Resistor_SMD:R_0805_2012Metric" V 7530 1950 50  0001 C CNN
+F 3 "~" H 7600 1950 50  0001 C CNN
+	1    7600 1950
+	1    0    0    -1
+$EndComp
+Wire Wire Line
+	7600 1700 7600 1800
+Wire Wire Line
+	7600 1400 7600 1275
+Wire Wire Line
+	7600 1275 8050 1275
+Wire Wire Line
+	7600 1275 7425 1275
+Connection ~ 7600 1275
+Wire Wire Line
+	7600 2100 7600 2175
+Wire Wire Line
+	7600 2175 8050 2175
+Connection ~ 8050 2175
+Wire Wire Line
+	2100 2850 2875 2850
+Wire Wire Line
+	2100 4900 2875 4900
+Wire Wire Line
+	2100 750  2875 750
+Wire Wire Line
+	2100 750  1300 750
+Connection ~ 2100 750
+Wire Wire Line
+	2100 750  2100 700
+$Comp
+L power:+BATT #PWR0104
+U 1 1 601B4594
+P 2100 700
+F 0 "#PWR0104" H 2100 550 50  0001 C CNN
+F 1 "+BATT" H 2100 875 50  0000 C CNN
+F 2 "" H 2100 700 50  0001 C CNN
+F 3 "" H 2100 700 50  0001 C CNN
+	1    2100 700
+	1    0    0    -1
+$EndComp
 $EndSCHEMATC
