File: RADSAT-SK Timer/RADSAT-SK Timer.sch (KiCad schematic (older format))
At the start: 73 parts, among them J101 Conn_02x26_Odd_Even, J103 Conn_02x26_Odd_Even, Q101 IRLML2060, Q102 IRLML2060, Q103 IRLML2060, Q104 IRLML2060, Q105 IRLML2060, Q106 IRLML2060, Q107 IRLML2060, Q108 IRLML2060, Q109 IRLML2060, U101 LM397MF, U102 LM397MF, U103 LM397MF, U104 CD4052B

Commit message: Deleted a bunch of backups and unnecessary project files
Parts:
- Q101, Q102, Q103, Q104, Q105, Q106, Q107, Q108, Q109: symbol RADSAT-SK-Timer-rescue:IRLML2060-Transistor_FET -> Transistor_FET:IRLML2060
- U101, U102, U103: symbol RADSAT-SK-Timer-rescue:LM397MF-LM397MF -> LM397MF:LM397MF
- U104: symbol RADSAT-SK-Timer-rescue:CD4052B-Analog_Switch -> Analog_Switch:CD4052B
Changed lines of the file:
@@
 EESchema Schematic File Version 4
-LIBS:RADSAT-SK Timer-cache
-EELAYER 26 0
+EELAYER 30 0
 EELAYER END
 $Descr A4 11693 8268
@@
 $EndComp
 $Comp
-L RADSAT-SK-Timer-rescue:CD4052B-Analog_Switch U104
+L Analog_Switch:CD4052B U104
 U 1 1 5FF9C3C1
 P 9125 1475
@@
 Wire Wire Line
 	8050 1675 8050 2175
-$Comp
-L power:+BATT #PWR0104
-U 1 1 601B4594
-P 2100 700
-F 0 "#PWR0104" H 2100 550 50  0001 C CNN
-F 1 "+BATT" H 2100 875 50  0000 C CNN
-F 2 "" H 2100 700 50  0001 C CNN
-F 3 "" H 2100 700 50  0001 C CNN
-	1    2100 700
-	1    0    0    -1
-$EndComp
 Wire Wire Line
 	9975 775  10625 775
@@
 Text Notes 7150 2675 0    79   ~ 0
 CSKB Connectors
-Wire Wire Line
-	2100 750  2100 700
-Connection ~ 2100 750
-Wire Wire Line
-	2100 750  1300 750
 Text Notes 525  6925 0    79   ~ 0
 Batteries, Charger, Booster, Mechanical Inhibits, Antenna Connector, Output Connectors
 $Comp
-L RADSAT-SK-Timer-rescue:IRLML2060-Transistor_FET Q104
+L Transistor_FET:IRLML2060 Q104
 U 1 1 600624B3
 P 1800 1525
@@
 $EndComp
 $Comp
-L RADSAT-SK-Timer-rescue:IRLML2060-Transistor_FET Q107
+L Transistor_FET:IRLML2060 Q107
 U 1 1 600655A8
 P 4300 1875
@@
 $EndComp
 $Comp
-L RADSAT-SK-Timer-rescue:IRLML2060-Transistor_FET Q101
+L Transistor_FET:IRLML2060 Q101
 U 1 1 6005D75A
 P 1200 1725
@@
 	600  750  600  1725
 $Comp
-L RADSAT-SK-Timer-rescue:LM397MF-LM397MF U101
+L LM397MF:LM397MF U101
 U 1 1 600CAF9B
 P 5525 1250
@@
 	2100 2850 1300 2850
 $Comp
-L RADSAT-SK-Timer-rescue:IRLML2060-Transistor_FET Q105
+L Transistor_FET:IRLML2060 Q105
 U 1 1 6023BB16
 P 1800 3625
@@
 $EndComp
 $Comp
-L RADSAT-SK-Timer-rescue:IRLML2060-Transistor_FET Q108
+L Transistor_FET:IRLML2060 Q108
 U 1 1 6023BB1C
 P 4300 3975
@@
 $EndComp
 $Comp
-L RADSAT-SK-Timer-rescue:IRLML2060-Transistor_FET Q102
+L Transistor_FET:IRLML2060 Q102
 U 1 1 6023BB2E
 P 1200 3825
@@
 	600  2850 600  3825
 $Comp
-L RADSAT-SK-Timer-rescue:LM397MF-LM397MF U102
+L LM397MF:LM397MF U102
 U 1 1 6023BB41
 P 5525 3350
@@
 	2100 4900 1300 4900
 $Comp
-L RADSAT-SK-Timer-rescue:IRLML2060-Transistor_FET Q106
+L Transistor_FET:IRLML2060 Q106
 U 1 1 60268B09
 P 1800 5675
@@
 $EndComp
 $Comp
-L RADSAT-SK-Timer-rescue:IRLML2060-Transistor_FET Q109
+L Transistor_FET:IRLML2060 Q109
 U 1 1 60268B0F
 P 4300 6025
@@
 $EndComp
 $Comp
-L RADSAT-SK-Timer-rescue:IRLML2060-Transistor_FET Q103
+L Transistor_FET:IRLML2060 Q103
 U 1 1 60268B21
 P 1200 5875
@@
 	600  4900 600  5875
 $Comp
-L RADSAT-SK-Timer-rescue:LM397MF-LM397MF U103
+L LM397MF:LM397MF U103
 U 1 1 60268B34
 P 5525 5400
@@
 Connection ~ 8050 2175
 Wire Wire Line
+	2100 2850 2875 2850
+Wire Wire Line
+	2100 4900 2875 4900
+Wire Wire Line
 	2100 750  2875 750
 Wire Wire Line
-	2100 2850 2875 2850
-Wire Wire Line
-	2100 4900 2875 4900
+	2100 750  1300 750
+Connection ~ 2100 750
+Wire Wire Line
+	2100 750  2100 700
+$Comp
+L power:+BATT #PWR0104
+U 1 1 601B4594
+P 2100 700
+F 0 "#PWR0104" H 2100 550 50  0001 C CNN
+F 1 "+BATT" H 2100 875 50  0000 C CNN
+F 2 "" H 2100 700 50  0001 C CNN
+F 3 "" H 2100 700 50  0001 C CNN
+	1    2100 700
+	1    0    0    -1
+$EndComp
 $EndSCHEMATC
