File: RADSAT-SK_timer_2/RADSAT-SK Timer 2.kicad_pcb (KiCad board)
At the start: 2 copper layers, 90.2 x 95.9 mm, 70 parts, among them J201 Conn_01x07, J202 Conn_01x05_Female, J203 Conn_01x03, J204 Conn_01x02, J205 Conn_01x02, J206 Conn_01x02, J207 Conn_02x26_Odd_Even, J208 Conn_02x26_Odd_Even, Q204 IRLML2060, Q205 IRLML2060, Q206 IRLML2060, SW201 SW_Push, SW202 SW_Push, SW203 SW_Push, SW204 SW_Push, SW205 SW_Push, SW206 SW_Push, U101 LT1521, U102 Galaxia_Timer, U202 TPS3700DDCR, U230 CPC1114N, U240 CPC1114N, U250 CPC1114N, U260 CPC1114N

Commit message: 555 push for production
Parts:
- removed TP111, TP112, TP113, TP114, TP115: TestPoint, S2761-46R:HARWIN_S2761-46R
- removed U102: Galaxia_Timer, Galaxia_Timer:Galaxia_Timer
- removed U202: TPS3700DDCR, Package_TO_SOT_SMD:TSOT-23-6
- added C104: 600uF, Capacitor_SMD:C_1206_3216Metric, F.Cu at (64.9, 99.4)
- added D101: SBR80520LT1G, Diode_SMD:D_SOD-123, F.Cu at (81.4, 71.6)
- added Q101: 2N7002E, Package_TO_SOT_SMD:SOT-23, F.Cu at (71.4, 84.0)
- added Q102: DSS4240T-7, Package_TO_SOT_SMD:SOT-23, F.Cu at (58.6, 100.7)
- added R112: 0, Resistor_SMD:R_1206_3216Metric_Pad1.30x1.75mm_HandSolder, F.Cu at (61.7, 87.9)
- added R113: 0, Resistor_SMD:R_1206_3216Metric_Pad1.30x1.75mm_HandSolder, F.Cu at (53.0, 98.9)
- added REF**: ESD-Logo_6.6x6mm_SilkScreen, Symbol:ESD-Logo_6.6x6mm_SilkScreen, F.Cu at (40.1, 99.6)
- C101: value 0.1uF -> 10nF; footprint Capacitor_SMD:C_0805_2012Metric -> Capacitor_SMD:C_1206_3216Metric
- C102: value 1uF -> 600uF; footprint Capacitor_SMD:C_0805_2012Metric -> Capacitor_SMD:C_1206_3216Metric
- C103: value 10uF -> 600uF; footprint Capacitor_SMD:C_0805_2012Metric -> Capacitor_SMD:C_1206_3216Metric
- D102: value RB751V40T1G -> SBR80520LT1G; footprint Diode_SMD:D_SOD-323 -> Diode_SMD:D_SOD-123
- R101: footprint Resistor_SMD:R_0805_2012Metric -> Resistor_SMD:R_1206_3216Metric_Pad1.30x1.75mm_HandSolder
- R102: value 604K -> 3M; footprint Resistor_SMD:R_0805_2012Metric -> Resistor_SMD:R_1206_3216Metric_Pad1.30x1.75mm_HandSolder
- R103: value 1k -> 1M; footprint Resistor_SMD:R_0805_2012Metric -> Resistor_SMD:R_1206_3216Metric_Pad1.30x1.75mm_HandSolder
- R104: value 2k -> 0; footprint Resistor_SMD:R_0805_2012Metric -> Resistor_SMD:R_1206_3216Metric_Pad1.30x1.75mm_HandSolder
- R105: value 49.9k -> 0; footprint Resistor_SMD:R_0805_2012Metric -> Resistor_SMD:R_1206_3216Metric_Pad1.30x1.75mm_HandSolder
- R107: value 81 -> 0; footprint Resistor_SMD:R_0805_2012Metric -> Resistor_SMD:R_1206_3216Metric_Pad1.30x1.75mm_HandSolder
- R108: value 100k -> 3M; footprint Resistor_SMD:R_0805_2012Metric -> Resistor_SMD:R_1206_3216Metric_Pad1.30x1.75mm_HandSolder
- R110: value 60 -> 40
- R111: value 17 -> 0; footprint Resistor_THT:R_Axial_DIN0309_L9.0mm_D3.2mm_P12.70mm_Horizontal -> Resistor_SMD:R_1206_3216Metric_Pad1.30x1.75mm_HandSolder
- R212, R214, R216: value 80 -> 260
- U101: value LT1521 -> TLC555CDR; footprint LT1521IS8-5TR:SO-8_S -> Package_SO:SOIC-8_3.9x4.9mm_P1.27mm
- moved R111 43.2 mm to (82.7, 78.5)
- moved R104 40.2 mm to (84.1, 97.6), turned to 0 degrees
- moved R108 33.8 mm to (59.2, 106.4), turned to 90 degrees
- moved U101 29.4 mm to (79.1, 85.2)
- moved D102 28.9 mm to (78.2, 100.3), turned to 270 degrees
- moved R107 28.5 mm to (83.9, 93.9)
- moved R101 28.3 mm to (72.4, 89.5), turned to 270 degrees
- moved R105 26.7 mm to (61.8, 103.8), turned to 270 degrees
- moved R103 26.2 mm to (65.6, 84.1), turned to 180 degrees
- moved R102 25.8 mm to (84.8, 84.0), turned to 270 degrees
- moved C102 23.0 mm to (84.8, 89.1)
- moved C103 15.5 mm to (68.7, 99.4), turned to 270 degrees
- moved C101 14.8 mm to (79.2, 90.2), turned to 180 degrees
Connections:
- C101 pad 1: +5V -> Net-(C101-Pad1)
- C102 pad 1: +5V -> Net-(C102-Pad1)
- C103 pad 2: GND -> Net-(C103-Pad2)
- D102 pad 2: Net-(C103-Pad1) -> Net-(D102-Pad2)
- D204 pad 1: B -> +BATT
- J203 pad 3: (no net) -> Net-(J203-Pad3)
- J207 pad 1: (no net) -> Net-(J207-Pad1)
- J207 pad 10: (no net) -> Net-(J207-Pad10)
- J207 pad 11: (no net) -> Net-(J207-Pad11)
- J207 pad 12: (no net) -> Net-(J207-Pad12)
- J207 pad 13: (no net) -> Net-(J207-Pad13)
- J207 pad 14: (no net) -> Net-(J207-Pad14)
- J207 pad 15: (no net) -> Net-(J207-Pad15)
- J207 pad 16: (no net) -> Net-(J207-Pad16)
- J207 pad 17: (no net) -> Net-(J207-Pad17)
- J207 pad 18: (no net) -> Net-(J207-Pad18)
- J207 pad 19: (no net) -> Net-(J207-Pad19)
- J207 pad 2: (no net) -> Net-(J207-Pad2)
- J207 pad 20: (no net) -> Net-(J207-Pad20)
- J207 pad 21: (no net) -> Net-(J207-Pad21)
- J207 pad 22: (no net) -> Net-(J207-Pad22)
- J207 pad 23: (no net) -> Net-(J207-Pad23)
- J207 pad 24: (no net) -> Net-(J207-Pad24)
- J207 pad 3: (no net) -> Net-(J207-Pad3)
- J207 pad 31: (no net) -> Net-(J207-Pad31)
- J207 pad 33: (no net) -> Net-(J207-Pad33)
- J207 pad 34: (no net) -> Net-(J207-Pad34)
- J207 pad 35: (no net) -> Net-(J207-Pad35)
- J207 pad 36: (no net) -> Net-(J207-Pad36)
- J207 pad 37: (no net) -> Net-(J207-Pad37)
- J207 pad 38: (no net) -> Net-(J207-Pad38)
- J207 pad 39: (no net) -> Net-(J207-Pad39)
- J207 pad 4: (no net) -> Net-(J207-Pad4)
- J207 pad 40: (no net) -> Net-(J207-Pad40)
- J207 pad 41: (no net) -> Net-(J207-Pad41)
- J207 pad 42: (no net) -> Net-(J207-Pad42)
- J207 pad 43: (no net) -> Net-(J207-Pad43)
- J207 pad 44: (no net) -> Net-(J207-Pad44)
- J207 pad 45: (no net) -> Net-(J207-Pad45)
- J207 pad 46: (no net) -> Net-(J207-Pad46)
- J207 pad 47: (no net) -> Net-(J207-Pad47)
- J207 pad 48: (no net) -> Net-(J207-Pad48)
- J207 pad 49: (no net) -> Net-(J207-Pad49)
- J207 pad 5: (no net) -> Net-(J207-Pad5)
- J207 pad 50: (no net) -> Net-(J207-Pad50)
- J207 pad 51: (no net) -> Net-(J207-Pad51)
- J207 pad 52: (no net) -> Net-(J207-Pad52)
- J207 pad 6: (no net) -> Net-(J207-Pad6)
- J207 pad 7: (no net) -> Net-(J207-Pad7)
- J207 pad 8: (no net) -> Net-(J207-Pad8)
- J207 pad 9: (no net) -> Net-(J207-Pad9)
- J208 pad 1: (no net) -> Net-(J208-Pad1)
- J208 pad 10: (no net) -> Net-(J208-Pad10)
- J208 pad 11: (no net) -> Net-(J208-Pad11)
- J208 pad 12: (no net) -> Net-(J208-Pad12)
- J208 pad 13: (no net) -> Net-(J208-Pad13)
- J208 pad 14: (no net) -> Net-(J208-Pad14)
- J208 pad 15: (no net) -> Net-(J208-Pad15)
- J208 pad 16: (no net) -> Net-(J208-Pad16)
- J208 pad 17: (no net) -> Net-(J208-Pad17)
- J208 pad 18: (no net) -> Net-(J208-Pad18)
- J208 pad 19: (no net) -> Net-(J208-Pad19)
- J208 pad 2: (no net) -> Net-(J208-Pad2)
- J208 pad 20: (no net) -> Net-(J208-Pad20)
- J208 pad 21: (no net) -> Net-(J208-Pad21)
- J208 pad 22: (no net) -> Net-(J208-Pad22)
- J208 pad 23: (no net) -> Net-(J208-Pad23)
- J208 pad 24: (no net) -> Net-(J208-Pad24)
- J208 pad 25: (no net) -> Net-(J208-Pad25)
- J208 pad 26: (no net) -> Net-(J208-Pad26)
- J208 pad 27: (no net) -> Net-(J208-Pad27)
- J208 pad 28: (no net) -> Net-(J208-Pad28)
- J208 pad 29: (no net) -> Net-(J208-Pad29)
- J208 pad 3: (no net) -> Net-(J208-Pad3)
- J208 pad 30: (no net) -> Net-(J208-Pad30)
- J208 pad 31: (no net) -> USB_Charge
- J208 pad 32: USB_Charge -> Net-(J208-Pad32)
- J208 pad 33: (no net) -> Net-(J208-Pad33)
- J208 pad 34: (no net) -> Net-(J208-Pad34)
- J208 pad 35: (no net) -> Net-(J208-Pad35)
- J208 pad 36: (no net) -> Net-(J208-Pad36)
- J208 pad 37: (no net) -> Net-(J208-Pad37)
- J208 pad 38: (no net) -> Net-(J208-Pad38)
- J208 pad 39: (no net) -> Net-(J208-Pad39)
- J208 pad 4: (no net) -> Net-(J208-Pad4)
- J208 pad 40: (no net) -> Net-(J208-Pad40)
- J208 pad 41: I2C_DATA -> Net-(J208-Pad41)
- J208 pad 42: (no net) -> I2C_DATA
- J208 pad 43: I2C_CLK -> Net-(J208-Pad43)
- J208 pad 44: (no net) -> I2C_CLK
- J208 pad 45: (no net) -> Net-(J208-Pad45)
- J208 pad 46: (no net) -> Net-(J208-Pad46)
- J208 pad 47: (no net) -> Net-(J208-Pad47)
- J208 pad 48: (no net) -> Net-(J208-Pad48)
- J208 pad 49: (no net) -> Net-(J208-Pad49)
- J208 pad 5: (no net) -> Net-(J208-Pad5)
- J208 pad 50: (no net) -> Net-(J208-Pad50)
- J208 pad 51: (no net) -> Net-(J208-Pad51)
- J208 pad 52: (no net) -> Net-(J208-Pad52)
- J208 pad 6: (no net) -> Net-(J208-Pad6)
- J208 pad 7: (no net) -> Net-(J208-Pad7)
- J208 pad 8: (no net) -> Net-(J208-Pad8)
- J208 pad 9: (no net) -> Net-(J208-Pad9)
- R101 pad 1: +5V -> Inhib_EN
- R101 pad 2: CHRG_ON-OFF -> GND
- R102 pad 1: Net-(R102-Pad1) -> Net-(D102-Pad1)
- R102 pad 2: B -> Net-(C102-Pad1)
- R103 pad 1: Net-(C103-Pad1) -> Net-(Q101-Pad3)
- R103 pad 2: Net-(R103-Pad2) -> Net-(D102-Pad1)
- R104 pad 1: Net-(R103-Pad2) -> Net-(D102-Pad2)
- R104 pad 2: GND -> +BATT
- R105 pad 1: Net-(R105-Pad1) -> Net-(C103-Pad2)
- R105 pad 2: Net-(R102-Pad1) -> GND
- R107 pad 1: A -> Net-(C103-Pad1)
- R107 pad 2: Net-(D102-Pad1) -> +BATT
- R108 pad 1: GND -> Net-(C103-Pad2)
- R108 pad 2: Net-(R105-Pad1) -> Net-(Q102-Pad1)
- R111 pad 1: GND -> Net-(D102-Pad1)
- R111 pad 2: Net-(D102-Pad1) -> Inhib_EN
- SW201 pad 2: B -> +BATT
- SW202 pad 2: B -> +BATT
- TP101 pad 1: B -> +BATT
- TP108 pad 1: I2C_DATA -> I2C_CLK
- TP110 pad 1: I2C_CLK -> I2C_DATA
- U101 pad 1: Net-(C103-Pad1) -> GND
- U101 pad 2: Net-(R103-Pad2) -> GND
- U101 pad 3: GND -> Net-(Q101-Pad1)
- U101 pad 4: (no net) -> Net-(D102-Pad1)
- U101 pad 5: CHRG_ON-OFF -> Net-(C101-Pad1)
- U101 pad 6: GND -> Net-(C102-Pad1)
- U101 pad 7: GND -> Net-(C102-Pad1)
- U101 pad 8: +5V -> Net-(D102-Pad1)
Routing:
- net B: track 116.1 -> 0.00 mm, vias 1 -> 0
- net Inhib_EN: track 10.6 -> 80.9 mm
- net +BATT: track 0.00 -> 54.5 mm, vias 0 -> 1
- net Net-(Q206-Pad3): track 136.6 -> 88.3 mm
- net CHRG_ON-OFF: track 41.6 -> 0.00 mm
- net +5V: track 156.2 -> 117.3 mm
- net Net-(R105-Pad1): track 21.2 -> 0.00 mm
- net USB_Charge: track 36.4 -> 57.2 mm
- net Net-(D102-Pad1): track 22.4 -> 40.5 mm
- net I2C_CLK: track 83.2 -> 68.1 mm
- net Net-(Q204-Pad3): track 118.9 -> 133.3 mm
- net Net-(C103-Pad2): track 0.00 -> 14.2 mm
- net Net-(R103-Pad2): track 14.1 -> 0.00 mm
- net Net-(D204-Pad6): track 51.4 -> 65.2 mm, vias 0 -> 1
- net Net-(R102-Pad1): track 13.7 -> 0.00 mm
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Other:
- net class Power added: clearance 0.2, trace_width 0.6, via_dia 0.8, via_drill 0.4
- board text added: "."
- board text added: "1"
- board text added: "4"
- board text added: "5"
- board text added: "555 Timer"
- board text added: "555 and RC 30 Minute Timer Proof of Concept Designed By : Atharva Parag Kulkarni Date: 6th February, 2023 Rev A"
- board text added: "8"
- board text added: "Caps, Diodes and Hope"
- board text added: "For 555: Desolder R113, 107 and solder R104, 112, 111, 101 For RC: Desolder R101, R104, 112, 111 and solder R113, 107"
- board text added: "RC Timer"
- board text removed: "Canadian Space Agency"
- board text removed: "Luc Charbonneau Lucus Rowlands"
- board text removed: "Project Made Possible By Don Seaman Joseph Remai Don Listwin Mark Teed"
